Commit message: Updated urdf for ur5e.
	1. Updated joint names.
	2. Fixed paths for mesh files.

File: urdf/ur5e/ur5e.urdf (robot description, URDF)
Before this commit: robot ur5e, 12 links, 11 joints
Links:
- removed link tool_handle
- removed link tool_tip
- added link tool_handle_link
- added link tool_tip_link
- link articulated_joint_link: geometry visual mesh filename=file://./meshes/ur5e/joint_tip.STL scale=0.001 0.001 0.001
- link base_link: geometry visual mesh filename=file://./meshes/ur5e/base.dae
- link link1: geometry visual mesh filename=file://./meshes/ur5e/shoulder.dae
- link link2: geometry visual mesh filename=file://./meshes/ur5e/upperarm.dae
- link link3: geometry visual mesh filename=file://./meshes/ur5e/forearm.dae
- link link4: geometry visual mesh filename=file://./meshes/ur5e/wrist1.dae
- link link5: geometry visual mesh filename=file://./meshes/ur5e/wrist2.dae
- link link6: geometry visual mesh filename=file://./meshes/ur5e/ee-and-drill-mesh-Demo-0228-Chen-cad-i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 scale=1 1 1
Joints:
- removed joint articulated_joint
- added joint tool_articulated_joint: type revolute, parent link6, child articulated_joint_link, origin xyz=0 -0.1696 0.2456 rpy=0 -1.5708 0.0, axis 0 0 1, limit lower=0.0001 upper=0.7845 effort=10 velocity=1
- joint handle_fixed_joint: child tool_handle -> tool_handle_link
- joint tip_joint: child tool_tip -> tool_tip_link

Commit message: Update path for mesh files, changed from "file://." to "../..".

File: urdf/ur5e/ur5e.urdf (robot description, URDF)
Before this commit: robot ur5e, 12 links, 11 joints
Links:
- link articulated_joint_link: geometry visual mesh filename=../../meshes/ur5e/joint_tip.STL scale=0.001 0.001 0.001
- link base_link: geometry visual mesh filename=../../meshes/ur5e/base.dae
- link link1: geometry visual mesh filename=../../meshes/ur5e/shoulder.dae
- link link2: geometry visual mesh filename=../../meshes/ur5e/upperarm.dae
- link link3: geometry visual mesh filename=../../meshes/ur5e/forearm.dae
- link link4: geometry visual mesh filename=../../meshes/ur5e/wrist1.dae
- link link5: geometry visual mesh filename=../../meshes/ur5e/wrist2.dae
- link link6: geometry visual mesh filename=../../meshes/ur5e/ee-and-drill-mesh-Demo-0228-Chen-cad-in-m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 scale=1 1 1
