Commit message: Update urdf for uf850, sync with drill_2024, branch flipped-base-mounting.

File: urdf/uf850/uf850.urdf (robot description, URDF)
Before this commit: robot uf850_raad_alpha1p1c, 15 links, 14 joints
Links:
- removed link cnl_link
- removed link tool_handle
- removed link tool_shaft_link
- removed link tool_tip
- added link tool_handle_link, mass 0.059728; collision mesh filename=package://uf850_raad_alpha1p1b/meshes/tool_handle_link.STL; visual mesh filename=package://uf850_raad_alpha1p1b/meshes/tool_handle_link.STL
- added link tool_tip_link, mass 2.65E-05; collision mesh filename=package://uf850_raad_alpha1p1b/meshes/tool_tip_link.STL; visual mesh filename=package://uf850_raad_alpha1p1b/meshes/tool_tip_link.STL
- link base_link: mass 2.26934676030042 -> 2.2693; geometry collision mesh filename=package://uf850_raad_alpha1p1b/meshes/base_link.STL; visual mesh filename=package://uf850_raad_alpha1p1b/meshes/base_link.STL
- link ee_mnt_link: mass 0.201702921570291 -> 0.15544; geometry collision mesh filename=package://uf850_raad_alpha1p1b/meshes/ee_mnt_link.STL; visual mesh filename=package://uf850_raad_alpha1p1b/meshes/ee_mnt_link.STL
- link ft_sensor_link: mass 0.0250988287832202 -> 0.0250988287832203; geometry collision mesh filename=package://uf850_raad_alpha1p1b/meshes/ft_sensor_link.STL; visual mesh filename=package://uf850_raad_alpha1p1b/meshes/ft_sensor_link.STL
- link link1: mass 2.58250832372613 -> 2.5825; geometry collision mesh filename=package://uf850_raad_alpha1p1b/meshes/link1.STL; visual mesh filename=package://uf850_raad_alpha1p1b/meshes/link1.STL
- link link2: mass 3.92627963689085 -> 3.9263; geometry collision mesh filename=package://uf850_raad_alpha1p1b/meshes/link2.STL; visual mesh filename=package://uf850_raad_alpha1p1b/meshes/link2.STL
- link link3: mass 1.93939268353003 -> 1.93939268353005; geometry collision mesh filename=package://uf850_raad_alpha1p1b/meshes/link3.STL; visual mesh filename=package://uf850_raad_alpha1p1b/meshes/link3.STL
- link link4: mass 1.48547732134494 -> 1.4855; geometry collision mesh filename=package://uf850_raad_alpha1p1b/meshes/link4.STL; visual mesh filename=package://uf850_raad_alpha1p1b/meshes/link4.STL
- link link5: mass 0.789449785943745 -> 0.78944978594375; geometry collision mesh filename=package://uf850_raad_alpha1p1b/meshes/link5.STL; visual mesh filename=package://uf850_raad_alpha1p1b/meshes/link5.STL
- link link6: mass 0.141894683215408 -> 0.14189; geometry collision mesh filename=package://uf850_raad_alpha1p1b/meshes/link6.STL; visual mesh filename=package://uf850_raad_alpha1p1b/meshes/link6.STL
- link tool_head_link: mass 0.000815640913959618 -> 0.00049397; geometry collision mesh filename=package://uf850_raad_alpha1p1b/meshes/tool_head_link.STL; visual mesh filename=package://uf850_raad_alpha1p1b/meshes/tool_head_link.STL
- link tool_mnt_link: mass 0.169976238671358 -> 0.110626907130558; geometry collision mesh filename=package://uf850_raad_alpha1p1b/meshes/tool_mnt_link.STL; visual mesh filename=package://uf850_raad_alpha1p1b/meshes/tool_mnt_link.STL
Joints:
- removed joint articulated_joint
- removed joint cnl_fixed_joint
- removed joint tool_handle_joint
- removed joint tool_shaft_fixed_joint
- removed joint tool_tip_fixed_joint
- added joint tip_link_fixed_joint: type fixed, parent tool_head_link, child tool_tip_link, origin xyz=0.0174 0.014749 0 rpy=-1.5708 -1.5708 0, axis 0 0 0
- added joint tool_articulated_joint: type revolute, parent tool_handle_link, child tool_head_link, origin xyz=0 -0.01075 -0.2305 rpy=0 1.5708 0, axis 0 0 1, limit lower=0 upper=0.6981 effort=0 velocity=0
- added joint tool_handle_fixed_joint: type fixed, parent tool_mnt_link, child tool_handle_link, origin xyz=-0.0595 0 0.07975 rpy=-1.5708 0 1.5708, axis 0 0 0
- joint ee_mnt_fixed_joint: origin xyz=0 0 0.027 rpy=0 0 0 -> xyz=0 0 0.03 rpy=0 0 0
- joint ft_sensor_fixed_joint: origin xyz=0.0695 0 -0.025 rpy=0 -1.5708 3.1416 -> xyz=0 0.0695 -0.025 rpy=-1.5708 -1.5708 0
- joint joint1: origin xyz=0 0 0.1855 rpy=0 0 0 -> xyz=0 0 0.185 rpy=0 0 0
- joint joint2: origin xyz=0 -0.015 0.1785 rpy=0 -1.5708 1.5708 -> xyz=0 -0.015 0.1785 rpy=1.5708 -1.5708 0
- joint joint3: origin xyz=0.39 0 -0.045 rpy=-3.1416 0 -1.5708 -> xyz=0.39 0 -0.045 rpy=3.1416 0 -1.5708
- joint joint5: origin xyz=-2.0826E-05 -0.051 0.266 rpy=0 -1.5708 -1.5708 -> xyz=-2.0826E-05 -0.051 0.266 rpy=-1.5708 -1.5708 0
- joint tool_mnt_fixed_joint: origin xyz=0.0205 0 0.10725 rpy=0 -1.5708 3.1416 -> xyz=0 0 0.0095 rpy=0 0 0
